File: hardware/rome.kicad_sch (KiCad schematic)
At the start: 13 parts, among them U1 KM62256CLP, U2 74HC595, U3 74HC595, U4 74LS245, U5 74LS245, U6 74LS245, U7 74LS32

Commit message: update hardware schematic; minimal firmware implementation
Parts:
- added J1: DIN41612_02x16_AB, symbol Connector:DIN41612_02x16_AB
- U1: footprint Package_DIP:DIP-28_W15.24mm -> Package_DIP:DIP-32_W7.62mm; symbol Memory_RAM:KM62256CLP -> ram_lib:24257(24512)
Connections:
- net +5V: now also U1.30 (VCC(CS2)), U1.32 (VCC), J1.b1 (Pin_b1); no longer U1.28 (VCC)
- net Address0: now also U1.12 (A0); no longer U1.10 (A0)
- net Address1: now also U1.11 (A1); no longer U1.9 (A1)
- net Address10: now also U1.23 (A10); no longer U1.21 (A10)
- net Address11: now also U1.25 (A11); no longer U1.23 (A11)
- net Address12: now also U1.4 (A12); no longer U1.2 (A12)
- net Address13: now also U1.28 (A13); no longer U1.26 (A13)
- net Address14: now also U1.3 (A14); no longer U1.1 (A14)
- net Address2: now also U1.10 (A2); no longer U1.8 (A2)
- net Address3: now also U1.9 (A3); no longer U1.7 (A3)
- net Address4: now also U1.8 (A4); no longer U1.6 (A4)
- net Address5: now also U1.7 (A5); no longer U1.5 (A5)
- net Address6: now also U1.6 (A6); no longer U1.4 (A6)
- net Address7: now also U1.5 (A7); no longer U1.3 (A7)
- net Address8: now also U1.27 (A8); no longer U1.25 (A8)
- net Address9: now also U1.26 (A9); no longer U1.24 (A9)
- net Data0: now also U1.13 (Q0); no longer U1.11 (Q0)
- net Data1: now also U1.14 (Q1); no longer U1.12 (Q1)
- net Data2: now also U1.15 (Q2); no longer U1.13 (Q2)
- net Data3: now also U1.17 (Q3); no longer U1.15 (Q3)
- net Data4: now also U1.18 (Q4); no longer U1.16 (Q4)
- net Data5: now also U1.19 (Q5); no longer U1.17 (Q5)
- net Data6: now also U1.20 (Q6); no longer U1.18 (Q6)
- net Data7: now also U1.21 (Q7); no longer U1.19 (Q7)
- net GND: now also U1.22 (~{CS}/~{CS1}), J1.a16 (Pin_a16); no longer U1.20 (~{CS})
- net ~{ECS}: now also J1.b11 (Pin_b11)
- net ~{ER}: now also J1.b9 (Pin_b9)
- net ~{EW}: now also J1.b4 (Pin_b4)
- net ~{IntRead}: now also U1.24 (~{OE}); no longer U1.22 (~{OE})
- net ~{IntWrite}: now also U1.29 (~{WE}); no longer U1.27 (~{WE})
- net Address15: now reaches U3.7 (QH)
- net Address15: now also U1.31 ((A15)), U6.11 (B7)
- net EAddress0: now reaches U5.2 (A0)
- net EAddress0: now also J1.a12 (Pin_a12)
- net EAddress1: now reaches U5.3 (A1)
- net EAddress1: now also J1.a11 (Pin_a11)
- net EAddress2: now reaches U5.4 (A2)
- net EAddress2: now also J1.a10 (Pin_a10)
- net EAddress3: now reaches U5.5 (A3)
- net EAddress3: now also J1.a9 (Pin_a9)
- net EAddress4: now reaches U5.6 (A4)
- net EAddress4: now also J1.a8 (Pin_a8)
- net EAddress5: now reaches U5.7 (A5)
- net EAddress5: now also J1.a7 (Pin_a7)
- net EAddress6: now reaches U5.8 (A6)
- net EAddress6: now also J1.a6 (Pin_a6)
- net EAddress7: now reaches U5.9 (A7)
- net EAddress7: now also J1.a5 (Pin_a5)
- net EAddress8: now reaches U6.2 (A0)
- net EAddress8: now also J1.b6 (Pin_b6)
- net EAddress9: now reaches U6.3 (A1)
- net EAddress9: now also J1.b7 (Pin_b7)
- net EAddress10: now reaches U6.4 (A2)
- net EAddress10: now also J1.b10 (Pin_b10)
- net EAddress11: now reaches U6.5 (A3)
- net EAddress11: now also J1.b8 (Pin_b8)
- net EAddress12: now reaches U6.6 (A4)
- net EAddress12: now also J1.a4 (Pin_a4)
- net EAddress13: now reaches U6.7 (A5)
- net EAddress13: now also J1.b5 (Pin_b5)
- net EAddress14: now reaches U6.8 (A6)
- net EAddress14: now also J1.a3 (Pin_a3)
- net EAddress15: now reaches U6.9 (A7)
- net EAddress15: now also J1.b2 (Pin_b2)
- net EData0: now reaches U4.2 (A0)
- net EData0: now also J1.a13 (Pin_a13)
- net EData1: now reaches U4.3 (A1)
- net EData1: now also J1.a14 (Pin_a14)
- net EData2: now reaches U4.4 (A2)
- net EData2: now also J1.a15 (Pin_a15)
- net EData3: now reaches U4.5 (A3)
- net EData3: now also J1.b16 (Pin_b16)
- net EData4: now reaches U4.6 (A4)
- net EData4: now also J1.b15 (Pin_b15)
- net EData5: now reaches U4.7 (A5)
- net EData5: now also J1.b14 (Pin_b14)
- net EData6: now reaches U4.8 (A6)
- net EData6: now also J1.b13 (Pin_b13)
- net EData7: now reaches U4.9 (A7)
- net EData7: now also J1.b12 (Pin_b12)
- no-connect marks 0 -> 3
Other:
- moved on the sheet: U2
